File: PCB/I2C_IO.kicad_pcb (KiCad board)
At the start: 2 copper layers, 132.1 x 111.8 mm, 65 parts, among them J1 Conn_01x06, J10 Conn_01x08, J11 Conn_01x02, J12 Conn_01x01, J13 Conn_01x01, J14 Conn_01x01, J15 Conn_01x01, J16 Conn_01x04, J17 Conn_01x04, J2 Conn_01x06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

Commit message: Test programm und abblock kondensatoren
Routing:
- net /K1-12: track 27.7 -> 72.7 mm
- net /K8-12: track 27.0 -> 54.1 mm
- net /K2-12: track 28.1 -> 54.2 mm
- net /K5-12: track 25.9 -> 51.8 mm
- net /K7-12: track 29.1 -> 54.8 mm
- net /K6-12: track 25.6 -> 51.2 mm
- net /K4-12: track 25.4 -> 50.8 mm
- net /K3-12: track 25.1 -> 50.2 mm
- net /K8-11: track 22.9 -> 45.9 mm
- net /K7-11: track 23.2 -> 45.0 mm
- net /K6-11: track 21.5 -> 43.1 mm
- net /K1-11: track 21.1 -> 42.2 mm
- net /K3-11: track 20.9 -> 41.8 mm
- net /K2-11: track 20.6 -> 41.3 mm
- net /K4-11: track 20.6 -> 41.2 mm
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Other:
- board text added: "ESP-01/S"
- board text added: "Flash ESP"
- board text added: "GND; INTA; INTB GND; SDA; SCL GND; RXD; TXD"
- board text added: "Isolate"
- board text added: "MCP Adresse"
- board text added: "VCC GND SCL SDA"
