File: PCB/I2C_IO.sch (KiCad schematic (older format))
At the start: 65 parts, among them J1 Conn_01x06, J10 Conn_01x08, J11 Conn_01x02, J12 Conn_01x01, J13 Conn_01x01, J14 Conn_01x01, J15 Conn_01x01, J16 Conn_01x04, J17 Conn_01x04, J2 Conn_01x06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

Commit message: Test programm und abblock kondensatoren
Parts:
- added C? (x5): C, symbol Device:C
- added C?: CP, symbol Device:CP
- R1, R2, R3, R4, R5, R6, R7, R8: value R -> 330
- R10, R11, R14, R15, R16, R9: value R -> 10k
- R12, R13, R17, R18, R19, R20, R21, R22: value R -> 560
Connections:
- net +12V: now also C?.1, C?.1, C?.1
- net GND: now also C?.1, C?.2, C?.2, C?.2, C?.2, C?.2
- net VCC: now also C?.1, C?.1, C?.2
Changed lines of the file:
@@
 P 10050 5150
 F 0 "R10" V 10130 5150 50  0000 C CNN
-F 1 "R" V 10050 5150 50  0000 C CNN
+F 1 "10k" V 10050 5150 50  0000 C CNN
 F 2 "Resistors_THT:R_Axial_DIN0309_L9.0mm_D3.2mm_P12.70mm_Horizontal" V 9980 5150 50  0001 C CNN
 F 3 "" H 10050 5150 50  0001 C CNN
@@
 P 10250 5150
 F 0 "R11" V 10330 5150 50  0000 C CNN
-F 1 "R" V 10250 5150 50  0000 C CNN
+F 1 "10k" V 10250 5150 50  0000 C CNN
 F 2 "Resistors_THT:R_Axial_DIN0309_L9.0mm_D3.2mm_P12.70mm_Horizontal" V 10180 5150 50  0001 C CNN
 F 3 "" H 10250 5150 50  0001 C CNN
@@
 P 8350 4250
 F 0 "R9" V 8430 4250 50  0000 C CNN
-F 1 "R" V 8350 4250 50  0000 C CNN
+F 1 "10k" V 8350 4250 50  0000 C CNN
 F 2 "Resistors_THT:R_Axial_DIN0309_L9.0mm_D3.2mm_P12.70mm_Horizontal" V 8280 4250 50  0001 C CNN
 F 3 "" H 8350 4250 50  0001 C CNN
@@
 P 8450 5650
 F 0 "R14" V 8530 5650 50  0000 C CNN
-F 1 "R" V 8450 5650 50  0000 C CNN
+F 1 "10k" V 8450 5650 50  0000 C CNN
 F 2 "Resistors_THT:R_Axial_DIN0309_L9.0mm_D3.2mm_P12.70mm_Horizontal" V 8380 5650 50  0001 C CNN
 F 3 "" H 8450 5650 50  0001 C CNN
@@
 P 8700 5750
 F 0 "R15" V 8780 5750 50  0000 C CNN
-F 1 "R" V 8700 5750 50  0000 C CNN
+F 1 "10k" V 8700 5750 50  0000 C CNN
 F 2 "Resistors_THT:R_Axial_DIN0309_L9.0mm_D3.2mm_P12.70mm_Horizontal" V 8630 5750 50  0001 C CNN
 F 3 "" H 8700 5750 50  0001 C CNN
@@
 P 8450 5850
 F 0 "R16" V 8530 5850 50  0000 C CNN
-F 1 "R" V 8450 5850 50  0000 C CNN
+F 1 "10k" V 8450 5850 50  0000 C CNN
 F 2 "Resistors_THT:R_Axial_DIN0309_L9.0mm_D3.2mm_P12.70mm_Horizontal" V 8380 5850 50  0001 C CNN
 F 3 "" H 8450 5850 50  0001 C CNN
@@
 P 1350 900
 F 0 "R1" V 1430 900 50  0000 C CNN
-F 1 "R" V 1350 900 50  0000 C CNN
+F 1 "330" V 1350 900 50  0000 C CNN
 F 2 "Resistors_THT:R_Axial_DIN0309_L9.0mm_D3.2mm_P12.70mm_Horizontal" V 1280 900 50  0001 C CNN
 F 3 "" H 1350 900 50  0001 C CNN
@@
 P 3100 900
 F 0 "R2" V 3180 900 50  0000 C CNN
-F 1 "R" V 3100 900 50  0000 C CNN
+F 1 "330" V 3100 900 50  0000 C CNN
 F 2 "Resistors_THT:R_Axial_DIN0309_L9.0mm_D3.2mm_P12.70mm_Horizontal" V 3030 900 50  0001 C CNN
 F 3 "" H 3100 900 50  0001 C CNN
@@
 P 4800 900
 F 0 "R3" V 4880 900 50  0000 C CNN
-F 1 "R" V 4800 900 50  0000 C CNN
+F 1 "330" V 4800 900 50  0000 C CNN
 F 2 "Resistors_THT:R_Axial_DIN0309_L9.0mm_D3.2mm_P12.70mm_Horizontal" V 4730 900 50  0001 C CNN
 F 3 "" H 4800 900 50  0001 C CNN
@@
 P 6500 900
 F 0 "R4" V 6580 900 50  0000 C CNN
-F 1 "R" V 6500 900 50  0000 C CNN
+F 1 "330" V 6500 900 50  0000 C CNN
 F 2 "Resistors_THT:R_Axial_DIN0309_L9.0mm_D3.2mm_P12.70mm_Horizontal" V 6430 900 50  0001 C CNN
 F 3 "" H 6500 900 50  0001 C CNN
@@
 P 8200 900
 F 0 "R5" V 8280 900 50  0000 C CNN
-F 1 "R" V 8200 900 50  0000 C CNN
+F 1 "330" V 8200 900 50  0000 C CNN
 F 2 "Resistors_THT:R_Axial_DIN0309_L9.0mm_D3.2mm_P12.70mm_Horizontal" V 8130 900 50  0001 C CNN
 F 3 "" H 8200 900 50  0001 C CNN
@@
 P 3100 2650
 F 0 "R6" V 3180 2650 50  0000 C CNN
-F 1 "R" V 3100 2650 50  0000 C CNN
+F 1 "330" V 3100 2650 50  0000 C CNN
 F 2 "Resistors_THT:R_Axial_DIN0309_L9.0mm_D3.2mm_P12.70mm_Horizontal" V 3030 2650 50  0001 C CNN
 F 3 "" H 3100 2650 50  0001 C CNN
@@
 P 4800 2700
 F 0 "R7" V 4880 2700 50  0000 C CNN
-F 1 "R" V 4800 2700 50  0000 C CNN
+F 1 "330" V 4800 2700 50  0000 C CNN
 F 2 "Resistors_THT:R_Axial_DIN0309_L9.0mm_D3.2mm_P12.70mm_Horizontal" V 4730 2700 50  0001 C CNN
 F 3 "" H 4800 2700 50  0001 C CNN
@@
 P 6500 2700
 F 0 "R8" V 6580 2700 50  0000 C CNN
-F 1 "R" V 6500 2700 50  0000 C CNN
+F 1 "330" V 6500 2700 50  0000 C CNN
 F 2 "Resistors_THT:R_Axial_DIN0309_L9.0mm_D3.2mm_P12.70mm_Horizontal" V 6430 2700 50  0001 C CNN
 F 3 "" H 6500 2700 50  0001 C CNN
@@
 P 1400 5650
 F 0 "R12" V 1480 5650 50  0000 C CNN
-F 1 "R" V 1400 5650 50  0000 C CNN
+F 1 "560" V 1400 5650 50  0000 C CNN
 F 2 "Resistors_THT:R_Axial_DIN0309_L9.0mm_D3.2mm_P12.70mm_Horizontal" V 1330 5650 50  0001 C CNN
 F 3 "" H 1400 5650 50  0001 C CNN
@@
 P 1400 6200
 F 0 "R17" V 1480 6200 50  0000 C CNN
-F 1 "R" V 1400 6200 50  0000 C CNN
+F 1 "560" V 1400 6200 50  0000 C CNN
 F 2 "Resistors_THT:R_Axial_DIN0309_L9.0mm_D3.2mm_P12.70mm_Horizontal" V 1330 6200 50  0001 C CNN
 F 3 "" H 1400 6200 50  0001 C CNN
@@
 P 1400 6750
 F 0 "R19" V 1480 6750 50  0000 C CNN
-F 1 "R" V 1400 6750 50  0000 C CNN
+F 1 "560" V 1400 6750 50  0000 C CNN
 F 2 "Resistors_THT:R_Axial_DIN0309_L9.0mm_D3.2mm_P12.70mm_Horizontal" V 1330 6750 50  0001 C CNN
 F 3 "" H 1400 6750 50  0001 C CNN
@@
 P 1400 7300
 F 0 "R21" V 1480 7300 50  0000 C CNN
-F 1 "R" V 1400 7300 50  0000 C CNN
+F 1 "560" V 1400 7300 50  0000 C CNN
 F 2 "Resistors_THT:R_Axial_DIN0309_L9.0mm_D3.2mm_P12.70mm_Horizontal" V 1330 7300 50  0001 C CNN
 F 3 "" H 1400 7300 50  0001 C CNN
@@
 P 3400 5650
 F 0 "R13" V 3480 5650 50  0000 C CNN
-F 1 "R" V 3400 5650 50  0000 C CNN
+F 1 "560" V 3400 5650 50  0000 C CNN
 F 2 "Resistors_THT:R_Axial_DIN0309_L9.0mm_D3.2mm_P12.70mm_Horizontal" V 3330 5650 50  0001 C CNN
 F 3 "" H 3400 5650 50  0001 C CNN
@@
 P 3400 6200
 F 0 "R18" V 3480 6200 50  0000 C CNN
-F 1 "R" V 3400 6200 50  0000 C CNN
+F 1 "560" V 3400 6200 50  0000 C CNN
 F 2 "Resistors_THT:R_Axial_DIN0309_L9.0mm_D3.2mm_P12.70mm_Horizontal" V 3330 6200 50  0001 C CNN
 F 3 "" H 3400 6200 50  0001 C CNN
@@
 P 3400 6750
 F 0 "R20" V 3480 6750 50  0000 C CNN
-F 1 "R" V 3400 6750 50  0000 C CNN
+F 1 "560" V 3400 6750 50  0000 C CNN
 F 2 "Resistors_THT:R_Axial_DIN0309_L9.0mm_D3.2mm_P12.70mm_Horizontal" V 3330 6750 50  0001 C CNN
 F 3 "" H 3400 6750 50  0001 C CNN
@@
 P 3400 7300
 F 0 "R22" V 3480 7300 50  0000 C CNN
-F 1 "R" V 3400 7300 50  0000 C CNN
+F 1 "560" V 3400 7300 50  0000 C CNN
 F 2 "Resistors_THT:R_Axial_DIN0309_L9.0mm_D3.2mm_P12.70mm_Horizontal" V 3330 7300 50  0001 C CNN
 F 3 "" H 3400 7300 50  0001 C CNN
@@
 Wire Wire Line
 	5450 5650 5850 5650
+$Comp
+L Device:C C?
+U 1 1 5DB393BB
+P 2000 4300
+F 0 "C?" H 2115 4346 50  0000 L CNN
+F 1 "C" H 2115 4255 50  0000 L CNN
+F 2 "" H 2038 4150 50  0001 C CNN
+F 3 "~" H 2000 4300 50  0001 C CNN
+	1    2000 4300
+	1    0    0    -1
+$EndComp
+$Comp
+L Device:C C?
+U 1 1 5DB39AB4
+P 4950 4300
+F 0 "C?" H 5065 4346 50  0000 L CNN
+F 1 "C" H 5065 4255 50  0000 L CNN
+F 2 "" H 4988 4150 50  0001 C CNN
+F 3 "~" H 4950 4300 50  0001 C CNN
+	1    4950 4300
+	1    0    0    -1
+$EndComp
+Wire Wire Line
+	2000 4100 2000 4150
+Connection ~ 2000 4100
+Wire Wire Line
+	2000 4450 2000 4500
+Wire Wire Line
+	2000 4500 1550 4500
+Connection ~ 1550 4500
+Wire Wire Line
+	4950 4150 4750 4150
+$Comp
+L power:GND #PWR?
+U 1 1 5DBA7EE6
+P 4950 4500
+F 0 "#PWR?" H 4950 4250 50  0001 C CNN
+F 1 "GND" H 4950 4350 50  0000 C CNN
+F 2 "" H 4950 4500 50  0001 C CNN
+F 3 "" H 4950 4500 50  0001 C CNN
+	1    4950 4500
+	1    0    0    -1
+$EndComp
+Wire Wire Line
+	4950 4450 4950 4500
+$Comp
+L Device:C C?
+U 1 1 5DBCD367
+P 2250 2950
+F 0 "C?" H 2365 2996 50  0000 L CNN
+F 1 "C" H 2365 2905 50  0000 L CNN
+F 2 "" H 2288 2800 50  0001 C CNN
+F 3 "~" H 2250 2950 50  0001 C CNN
+	1    2250 2950
+	1    0    0    -1
+$EndComp
+$Comp
+L power:GND #PWR?
+U 1 1 5DBCE0F1
+P 2250 3150
+F 0 "#PWR?" H 2250 2900 50  0001 C CNN
+F 1 "GND" H 2250 3000 50  0000 C CNN
+F 2 "" H 2250 3150 50  0001 C CNN
+F 3 "" H 2250 3150 50  0001 C CNN
+	1    2250 3150
+	1    0    0    -1
+$EndComp
+Wire Wire Line
+	2250 3100 2250 3150
+Wire Wire Line
+	2250 2800 2250 2750
+Connection ~ 2250 2750
+$Comp
+L Device:C C?
+U 1 1 5DC1917D
+P 7900 4000
+F 0 "C?" V 7648 4000 50  0000 C CNN
+F 1 "C" V 7739 4000 50  0000 C CNN
+F 2 "" H 7938 3850 50  0001 C CNN
+F 3 "~" H 7900 4000 50  0001 C CNN
+	1    7900 4000
+	0    1    1    0
+$EndComp
+$Comp
+L power:GND #PWR?
+U 1 1 5DC1B65A
+P 8150 4000
+F 0 "#PWR?" H 8150 3750 50  0001 C CNN
+F 1 "GND" H 8150 3850 50  0000 C CNN
+F 2 "" H 8150 4000 50  0001 C CNN
+F 3 "" H 8150 4000 50  0001 C CNN
+	1    8150 4000
+	1    0    0    -1
+$EndComp
+Wire Wire Line
+	8050 4000 8150 4000
+Wire Wire Line
+	7600 4000 7750 4000
+Connection ~ 7600 4000
+$Comp
+L Device:C C?
+U 1 1 5DC67A3A
+P 1100 4300
+F 0 "C?" H 1215 4346 50  0000 L CNN
+F 1 "C" H 1215 4255 50  0000 L CNN
+F 2 "" H 1138 4150 50  0001 C CNN
+F 3 "~" H 1100 4300 50  0001 C CNN
+	1    1100 4300
+	1    0    0    -1
+$EndComp
+$Comp
+L Device:CP C?
+U 1 1 5DC68B2D
+P 750 4300
+F 0 "C?" H 868 4346 50  0000 L CNN
+F 1 "CP" H 868 4255 50  0000 L CNN
+F 2 "" H 788 4150 50  0001 C CNN
+F 3 "~" H 750 4300 50  0001 C CNN
+	1    750  4300
+	1    0    0    -1
+$EndComp
+Wire Wire Line
+	1100 4100 750  4100
+Wire Wire Line
+	750  4100 750  4150
+Connection ~ 1100 4100
+Wire Wire Line
+	1100 4150 1100 4100
+Wire Wire Line
+	1550 4500 1100 4500
+Wire Wire Line
+	750  4500 750  4450
+Wire Wire Line
+	1100 4500 1100 4450
+Connection ~ 1100 4500
+Wire Wire Line
+	1100 4500 750  4500
 $EndSCHEMATC
